File: Starter_AVR.kicad_pcb (KiCad board)
At the start: 2 copper layers, 90.5 x 67.5 mm, 48 parts, among them CON1 USB-MICRO-B, IC1 ATMEGA32-P, J2 SIL8, J3 SIL8, J4 SIL8, J5 SIL8, K1 BARREL, K2 CONN_3, K3 CONN_3, K4 CONN_3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

Commit message: added Changed files
Connections:
- D2 pad 1: /rxd -> /L1
- D4 pad 1: /txd -> /L2
- IC1 pad 18: /BL -> /L1
- IC1 pad 19: Net-(IC1-Pad19) -> /L2
- IC1 pad 20: Net-(IC1-Pad20) -> /BL
- J5 pad 5: /BL -> /L1
- J5 pad 6: Net-(IC1-Pad19) -> /L2
- J5 pad 7: Net-(IC1-Pad20) -> /BL
Routing:
- net /L1: track 0.00 -> 47.5 mm
- net /L2: track 0.00 -> 46.7 mm
- net Net-(IC1-Pad20): track 38.5 -> 0.00 mm
- net Net-(IC1-Pad19): track 26.0 -> 0.00 mm
- net /BL: track 46.9 -> 70.0 mm
- net /rxd: track 107.6 -> 96.1 mm
- net /txd: track 111.2 -> 101.2 mm
- net /S2: track 48.2 -> 55.5 mm
- added copper zone on F.Cu, net /+5V
- added copper zone on B.Cu, net GND
Other:
- net class Default: clearance 0.1778 -> 0.2286
- rule trace_clearance: 0.1778 -> 0.2286
- board text added: "B_LED"
