File: Starter_AVR.sch (KiCad schematic (older format))
At the start: 47 parts, among them CON1 USB-MICRO-B, IC1 ATMEGA32-P, J2 SIL8, J3 SIL8, J4 SIL8, J5 SIL8, K1 BARREL, K2 CONN_3, K3 CONN_3, K4 CONN_3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

Commit message: added Changed files
Connections:
- net BL: now also IC1.20 ((ICP)PD6), J5.7; no longer IC1.18 ((OC1B)PD4), J5.5
- net rxd: no longer D2.1 (A)
- net txd: no longer D4.1 (A)
- net L2: now reaches IC1.19 ((OC1A)PD5), J5.6
- net L2: now also D4.1 (A)
- new net L1: D2.1 (A), IC1.18 ((OC1B)PD4), J5.5
Changed lines of the file:
@@
 Text Label 10200 3750 0    60   ~ 0
 DRST
-Text Label 8000 6100 0    60   ~ 0
-rxd
-Text Label 8000 6350 0    60   ~ 0
-txd
 Text Label 7600 5450 0    60   ~ 0
 S1
@@
 $EndComp
 Text Label 8000 6600 0    60   ~ 0
-BL
-Text Label 4250 4500 0    60   ~ 0
 BL
 $Comp
@@
 Wire Wire Line
 	7450 3850 7450 3950
+Text Label 8000 6100 0    60   ~ 0
+L1
+Text Label 8000 6350 0    60   ~ 0
+L2
+Text Label 4250 4500 0    60   ~ 0
+L1
+Text Label 4250 4700 0    60   ~ 0
+BL
+Text Label 4250 4600 0    60   ~ 0
+L2
 $EndSCHEMATC
