File: Design Files/Starter_AVR.sch (KiCad schematic (older format))
At the start: 47 parts, among them CON1 USB-MICRO-B, IC1 ATMEGA32-P, J2 SIL8, J3 SIL8, J4 SIL8, J5 SIL8, K1 BARREL, K2 CONN_3, K3 CONN_3, K4 CONN_3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

Commit message: new design
Connections:
- net BL: now also IC1.20 ((ICP)PD6), J5.7; no longer IC1.18 ((OC1B)PD4), J5.5
- net GND: no longer CON1.5 (GND)
- net rxd: no longer D2.1 (A)
- net txd: no longer D4.1 (A)
- net L2: now reaches IC1.19 ((OC1A)PD5), J5.6
- net L2: now also D4.1 (A)
- new net L1: D2.1 (A), IC1.18 ((OC1B)PD4), J5.5
- no-connect marks 31 -> 32
Other:
- note added: "ADC Pot"
- moved on the sheet: C1, C2, CON1, D2, D4, D5, K1, P1, P2, P3, P4, P6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
